Commit message: feat: Finish integration gazebo sim & ros_control

File: msd700_description/urdf/common/materials.xacro (robot description, xacro)
@@ -7,3 +7,6 @@
         <color rgba="0 0 0 1"/>
     </material>
+    <material name="grey">
+        <color rgba="0.5 0.5 0.5 1"/>
+    </material>
 </robot>

File: msd700_description/urdf/common/wheel.urdf.xacro (robot description, xacro)
@@ -22,8 +22,10 @@
                 </geometry>
             </collision>
-            <xacro:cylinder_inertial m="1" r="${radius}" l="${thickness}" xyz="0 0 0" rpy="0 0 0"/>
+            <xacro:cylinder_inertial m="0.05" r="${radius}" l="${thickness}" xyz="0 0 0" rpy="0 0 0"/>
         </link>
         <gazebo reference="${prefix}_link">
             <material>Gazebo/Black</material>
+            <mu1>0.1</mu1>
+            <mu2>0.1</mu2>
         </gazebo>
     </xacro:macro>

File: msd700_description/urdf/gazebo/msd700_prototype.gazebo.xacro (robot description, xacro)
@@ -7,13 +7,4 @@
         </plugin>
     </gazebo>
-    <transmission name="fl_wheel_trans">
-        <type>transmission_interface/SimpleTransmission</type>
-        <actuator name="fl_wheel_motor">
-            <mechanicalReduction>1</mechanicalReduction>
-        </actuator>
-        <joint name="fl_wheel_joint">
-            <hardwareInterface>hardware_interface/VelocityJointInterface</hardwareInterface>
-        </joint>
-    </transmission>
     <transmission name="bl_wheel_trans">
         <type>transmission_interface/SimpleTransmission</type>
@@ -34,4 +25,13 @@
         </joint>
     </transmission>
+    <transmission name="fl_wheel_trans">
+        <type>transmission_interface/SimpleTransmission</type>
+        <actuator name="fl_wheel_motor">
+            <mechanicalReduction>1</mechanicalReduction>
+        </actuator>
+        <joint name="fl_wheel_joint">
+            <hardwareInterface>hardware_interface/VelocityJointInterface</hardwareInterface>
+        </joint>
+    </transmission>
     <transmission name="fr_wheel_trans">
         <type>transmission_interface/SimpleTransmission</type>

File: msd700_description/urdf/msd700_prototype.urdf.xacro (robot description, xacro)
@@ -1,17 +1,17 @@
 <?xml version="1.0"?>
 <robot xmlns:xacro="http://www.ros.org/wiki/xacro" name="msd700_prototype">
-    <xacro:property name="chassis_length" value="0.4"/>
-    <xacro:property name="chassis_width" value="0.3"/>
-    <xacro:property name="chassis_height" value="0.22"/>
+    <!-- Chassis Property -->
+    <xacro:property name="chassis_length" value="0.3"/>
+    <xacro:property name="chassis_width" value="0.2"/>
+    <xacro:property name="chassis_height" value="0.184"/>
+    <!-- Wheel Property -->
     <xacro:property name="wheel_radius" value="0.054"/>
     <xacro:property name="wheel_width" value="0.02"/>
+    <!-- Includes -->
     <xacro:include filename="$(find msd700_description)/urdf/common/inertials.xacro"/>
     <xacro:include filename="$(find msd700_description)/urdf/common/materials.xacro"/>
     <xacro:include filename="$(find msd700_description)/urdf/common/wheel.urdf.xacro"/>
     <xacro:include filename="$(find msd700_description)/urdf/sensors/2d_lidar.urdf.xacro"/>
-    <xacro:include filename="$(find msd700_description)/urdf/gazebo/msd700_prototype.gazebo.xacro"/>
-    <link name="base_link">
-        <!-- <origin xyz="0 0 ${chassis_height + wheel_radius/2}" rpy="0 0 0"/> -->
-    </link>
+    <link name="base_link" />
     <joint name="base_to_chassis_joint" type="fixed">
         <origin xyz="0 0 0" rpy="0 0 0"/>
@@ -21,27 +21,27 @@
     <link name="chassis_link">
         <visual>
-            <!-- <origin xyz="-${chassis_length/2} -${chassis_width/2} -${chassis_height/2}" rpy="0 0 0"/> -->
-            <origin xyz="-0.25 -0.15 -0.09" rpy="0 0 0"/>
+            <origin xyz="-0.15 -0.1 -0.092" rpy="0 0 0"/>
             <geometry>
-                <!-- <box size="${chassis_length} ${chassis_width} ${chassis_height}"/> -->
-                <mesh filename="package://msd700_description/meshes/msd700_without_arm.stl" scale="0.0015 0.0015 0.001"/>
+                <mesh filename="package://msd700_description/meshes/msd700_without_arm.stl" scale="0.001 0.001 0.001" />
             </geometry>
-            <material name="red"/>
+            <material name="grey"/>
         </visual>
         <collision>
             <origin xyz="0 0 0" rpy="0 0 0"/>
             <geometry>
-                <box size="${chassis_length} ${chassis_width} ${chassis_height}"/>
+                <box size="${chassis_length} ${chassis_width} ${chassis_height}" />
             </geometry>
         </collision>
-        <xacro:box_inertial m="10" w="${chassis_width}" l="${chassis_length}" d="${chassis_height}" xyz="0 0 0" rpy="0 0 0"/>
+        <xacro:box_inertial m="1" w="${chassis_width}" l="${chassis_length}" d="${chassis_height}" xyz="0 0 0" rpy="0 0 0"/>
     </link>
     <gazebo reference="chassis_link">
-        <material>Gazebo/Red</material>
+        <material>Gazebo/Grey</material>
     </gazebo>
-    <xacro:add_wheel prefix="fl_wheel" radius="${wheel_radius}" thickness="${wheel_width}" xyz="${chassis_length/2} ${chassis_width/2 + wheel_width/2} -${chassis_height/2}" parent="chassis_link"/>
-    <xacro:add_wheel prefix="fr_wheel" radius="${wheel_radius}" thickness="${wheel_width}" xyz="${chassis_length/2} -${chassis_width/2 + wheel_width/2} -${chassis_height/2}" parent="chassis_link"/>
+    <xacro:include filename="$(find msd700_description)/urdf/gazebo/msd700_prototype.gazebo.xacro"/>
     <xacro:add_wheel prefix="bl_wheel" radius="${wheel_radius}" thickness="${wheel_width}" xyz="-${chassis_length/2} ${chassis_width/2 + wheel_width/2} -${chassis_height/2}" parent="chassis_link"/>
     <xacro:add_wheel prefix="br_wheel" radius="${wheel_radius}" thickness="${wheel_width}" xyz="-${chassis_length/2} -${chassis_width/2 + wheel_width/2} -${chassis_height/2}" parent="chassis_link"/>
-    <xacro:add_2d_lidar prefix="lidar" topic="scan" parent="chassis_link" x="0" y="0" z="${chassis_height/2}" rpy="0 0 0"/>
+    <!-- <xacro:add_wheel prefix="mid_wheel" radius="${wheel_radius}" thickness="${wheel_width}" xyz="${chassis_length/2} 0 -${chassis_height/2}" parent="chassis_link"/> -->
+    <xacro:add_wheel prefix="fr_wheel" radius="${wheel_radius}" thickness="${wheel_width}" xyz="${chassis_length/2} -${chassis_width/2 + wheel_width/2} -${chassis_height/2}" parent="chassis_link"/>
+    <xacro:add_wheel prefix="fl_wheel" radius="${wheel_radius}" thickness="${wheel_width}" xyz="${chassis_length/2} ${chassis_width/2 + wheel_width/2} -${chassis_height/2}" parent="chassis_link"/>
+    <!-- <xacro:add_2d_lidar prefix="lidar" topic="scan" parent="chassis_link" x="0" y="0" z="${chassis_height/2}" rpy="0 0 0"/> -->
 </robot>

File: msd700_description/urdf/sensors/2d_lidar.urdf.xacro (robot description, xacro)
@@ -9,5 +9,5 @@
     <xacro:macro name="add_2d_lidar" params="prefix topic parent x y z rpy">
         <joint name="${prefix}_joint" type="fixed">
-            <origin xyz="${x} ${y} ${z+0.027}" rpy="${rpy}"/>
+            <origin xyz="${x} ${y} ${z+0.04}" rpy="${rpy}"/>
             <parent link="${parent}"/>
             <child link="${prefix}_link"/>
