Commit message: feat: fix simulation and clean up all namespace

File: msd700_description/urdf/common/wheel.urdf.xacro (robot description, xacro)
@@ -30,3 +30,31 @@
         </gazebo>
     </xacro:macro>
+    <xacro:macro name="add_caster_wheel" params="prefix radius thickness xyz parent">
+        <joint name="${prefix}_joint" type="fixed" >
+            <origin xyz="${xyz}" rpy="0 0 0"/>
+            <parent link="${parent}"/>
+            <child link="${prefix}_link"/>
+        </joint>
+        <link name="${prefix}_link">
+            <visual>
+                <origin xyz="0 0 0" rpy="-1.5708 0 0"/>
+                <geometry>
+                    <cylinder radius="${radius}" length="${thickness}"/>
+                </geometry>
+                <material name="black"/>
+            </visual>
+            <collision>
+                <origin xyz="0 0 0" rpy="-1.5708 0 0"/>
+                <geometry>
+                    <cylinder radius="${radius}" length="${thickness}"/>
+                </geometry>
+            </collision>
+            <xacro:cylinder_inertial m="0.05" r="${radius}" l="${thickness}" xyz="0 0 0" rpy="0 0 0"/>
+        </link>
+        <gazebo reference="${prefix}_link">
+            <material>Gazebo/Black</material>
+            <mu1>0.0</mu1>
+            <mu2>0.0</mu2>
+        </gazebo>
+    </xacro:macro>
 </robot>

File: msd700_description/urdf/msd700_prototype.urdf.xacro (robot description, xacro)
@@ -39,11 +39,9 @@
         <material>Gazebo/Grey</material>
     </gazebo>
-    <xacro:include filename="$(find msd700_description)/urdf/gazebo/msd700_prototype.gazebo.xacro"/>
+    <xacro:include filename="$(find msd700_description)/urdf/control/msd700_prototype_control.xacro"/>
     <xacro:add_wheel prefix="bl_wheel" radius="${wheel_radius}" thickness="${wheel_width}" xyz="-${chassis_length/2} ${chassis_width/2 + wheel_width/2} -${chassis_height/2}" parent="chassis_link"/>
     <xacro:add_wheel prefix="br_wheel" radius="${wheel_radius}" thickness="${wheel_width}" xyz="-${chassis_length/2} -${chassis_width/2 + wheel_width/2} -${chassis_height/2}" parent="chassis_link"/>
-    <!-- <xacro:add_wheel prefix="mid_wheel" radius="${wheel_radius}" thickness="${wheel_width}" xyz="${chassis_length/2} 0 -${chassis_height/2}" parent="chassis_link"/> -->
-    <xacro:add_wheel prefix="fr_wheel" radius="${wheel_radius}" thickness="${wheel_width}" xyz="${chassis_length/2} -${chassis_width/2 + wheel_width/2} -${chassis_height/2}" parent="chassis_link"/>
-    <xacro:add_wheel prefix="fl_wheel" radius="${wheel_radius}" thickness="${wheel_width}" xyz="${chassis_length/2} ${chassis_width/2 + wheel_width/2} -${chassis_height/2}" parent="chassis_link"/>
-    <xacro:add_2d_lidar prefix="lidar" topic="scan" parent="chassis_link" x="0" y="0" z="${chassis_height/2}" rpy="0 0 0"/>
-    <!-- <xacro:add_imu prefix="imu" topic="imu" parent="chassis_link" xyz="0 0 0.02" rpy="0 0 0"/> -->
+    <xacro:add_caster_wheel prefix="fl_wheel" radius="${wheel_radius}" thickness="${wheel_width}" xyz="${chassis_length/2} ${chassis_width/2 + wheel_width/2} -${chassis_height/2}" parent="chassis_link"/>
+    <xacro:add_caster_wheel prefix="fr_wheel" radius="${wheel_radius}" thickness="${wheel_width}" xyz="${chassis_length/2} -${chassis_width/2 + wheel_width/2} -${chassis_height/2}" parent="chassis_link"/>
+    <xacro:add_2d_lidar prefix="lidar" topic="/msd700/sensors/scan" parent="chassis_link" x="0" y="0" z="${chassis_height/2}" rpy="0 0 0"/>
 </robot>
